Commit message: Fixed typo that resulted in error of no visualization in Rviz and corrected wheel_right_link values to 90, to accurately position

File: install/bumperbot_description/share/bumperbot_description/urdf/bumperbot.urdf.xacro (robot description, xacro)
@@ -15,3 +15,17 @@
         <origin rpy="0 0 0" xyz="0 0 0.033" />
     </joint>
+    <link name="wheel_ride_link">
+        <visual>
+            <origin rpy="0 0 0" xyz="0 0 0" />
+            <geometry>
+                <mesh filename="package://bumperbot_description/meshes/wheel_right_link.STL" />
+            </geometry>
+        </visual>
+    </link>
+    <!-- <joint name="wheel_right_joint" type="continuous">
+        <parent link="base_link" />
+        <child link="wheel_right_link" />
+        <axis xyz="0 1 0" />
+        <origin rpy="0 0 0" xyz="0 -0.07 0" />
+    </joint> -->
 </robot>

File: src/bumperbot_description/urdf/bumperbot.urdf.xacro (robot description, xacro)
@@ -15,7 +15,7 @@
         <origin rpy="0 0 0" xyz="0 0 0.033" />
     </joint>
-    <link name="wheel_ride_link">
+    <link name="wheel_right_link">
         <visual>
-            <origin rpy="0 0 0" xyz="0 0 0" />
+            <origin rpy="1.57 0 0" xyz="0 0 0" />
             <geometry>
                 <mesh filename="package://bumperbot_description/meshes/wheel_right_link.STL" />

Commit message: Added Simple Parameter node in py

File: install/bumperbot_description/share/bumperbot_description/urdf/bumperbot.urdf.xacro (robot description, xacro)
@@ -15,7 +15,7 @@
         <origin rpy="0 0 0" xyz="0 0 0.033" />
     </joint>
-    <link name="wheel_ride_link">
+    <link name="wheel_right_link">
         <visual>
-            <origin rpy="0 0 0" xyz="0 0 0" />
+            <origin rpy="1.57 0 0" xyz="0 0 0" />
             <geometry>
                 <mesh filename="package://bumperbot_description/meshes/wheel_right_link.STL" />
@@ -23,9 +23,49 @@
         </visual>
     </link>
-    <!-- <joint name="wheel_right_joint" type="continuous">
+    <joint name="wheel_right_joint" type="continuous">
         <parent link="base_link" />
         <child link="wheel_right_link" />
         <axis xyz="0 1 0" />
         <origin rpy="0 0 0" xyz="0 -0.07 0" />
-    </joint> -->
+    </joint>
+    <link name="wheel_left_link">
+        <visual>
+            <origin rpy="-1.57 0 0" xyz="0 0 0" />
+            <geometry>
+                <mesh filename="package://bumperbot_description/meshes/wheel_left_link.STL" />
+            </geometry>
+        </visual>
+    </link>
+    <joint name="wheel_left_joint" type="continuous">
+        <parent link="base_link" />
+        <child link="wheel_left_link" />
+        <axis xyz="0 1 0" />
+        <origin rpy="0 0 0" xyz="0 0.07 0" />
+    </joint>
+    <link name="castor_front_link">
+        <visual>
+            <origin rpy="0 0 0" xyz="0 0 0" />
+            <geometry>
+                <mesh filename="package://bumperbot_description/meshes/castor_front_link.STL" />
+            </geometry>
+        </visual>
+    </link>
+    <joint name="castor_front_joint" type="fixed">
+        <parent link="base_link" />
+        <child link="castor_front_link" />
+        <origin rpy="0 0 0" xyz="0.04755 0 -0.0275" />
+    </joint>
+    <link name="castor_rear_link">
+        <visual>
+            <origin rpy="0 0 0" xyz="0 0 0" />
+            <geometry>
+                <mesh filename="package://bumperbot_description/meshes/castor_rear_link.STL" />
+            </geometry>
+        </visual>
+    </link>
+    <joint name="castor_rear_joint" type="fixed">
+        <parent link="base_link" />
+        <child link="castor_rear_link" />
+        <origin rpy="0 0 0" xyz="-0.04755 0 -0.0275" />
+    </joint>
 </robot>
